File: pll/pll.kicad_pcb (KiCad board)
At the start: 2 copper layers, 24 parts, among them SW1 SW_DIP_x05, U1 NE555, U2 74HC393, U3 74HC86, U4 LM7805, U5 NE555

Commit message: Update pll
Signed-off-by: Felipe Leon <fglfgl27@gmail.com>
Parts:
- moved D1 57.1 mm to (75.7, 68.1)
- moved R5 57.1 mm to (80.3, 80.8)
- moved R4 57.1 mm to (94.5, 62.0)
- moved R8 57.1 mm to (70.1, 88.4)
- moved RV1 57.1 mm to (113.8, 62.0)
- moved U3 57.1 mm to (87.4, 75.2)
- moved C1 57.1 mm to (49.8, 57.9)
- moved C2 57.1 mm to (61.5, 57.9)
- moved C3 57.1 mm to (69.1, 68.1)
- moved C4 57.1 mm to (79.8, 97.5)
- moved D2 57.1 mm to (56.9, 81.3)
- moved J_in1 57.1 mm to (43.1, 51.8)
- moved R1 57.1 mm to (87.4, 52.8)
- moved R10 57.1 mm to (26.4, 98.6)
- moved R3 57.1 mm to (102.1, 74.2)
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Connections:
- R1 pad 1: Net-(R1-Pad1) -> Net-(C3-Pad1)
- R7 pad 1: Net-(R7-Pad1) -> Net-(C5-Pad1)
- U1 pad 6: Net-(R1-Pad1) -> Net-(C3-Pad1)
- U5 pad 6: Net-(R7-Pad1) -> Net-(C5-Pad1)
Routing:
- net Net-(C5-Pad1): track 23.0 -> 50.9 mm, vias 0 -> 2
- net Net-(C3-Pad1): track 21.5 -> 42.5 mm, vias 0 -> 2
- net Net-(R7-Pad1): track 9.63 -> 0.00 mm
- net Net-(R1-Pad1): track 5.29 -> 0.00 mm
- net GND: track 341.1 -> 337.6 mm
- net (no net): track 0.00 -> 2.87 mm
- net /out_counter_2_4_8: vias 0 -> 2
