File: oscila_mag/oscila_mag.sch (KiCad schematic (older format))
At the start: 31 parts, among them Q1 BC548, U1 TC4420CPA, U2 TC4420CPA

Commit message: Update pcbs
Signed-off-by: fgl27 <fglfgl27@gmail.com>
Parts:
- L1, L2: value 50u -> 45.6u
Other:
- moved on the sheet: D9, J_in1, Q1, R10, R12
Changed lines of the file:
@@
 P 6650 3450
 F 0 "L1" V 6650 3665 50  0000 C CNN
-F 1 "50u" V 6500 3700 50  0000 C CNN
+F 1 "45.6u" V 6500 3700 50  0000 C CNN
 F 2 "Inductor_THT:L_Toroid_Horizontal_D12.7mm_P20.00mm_Diameter14-5mm_Amidon-T50" H 6650 3450 50  0001 C CNN
 F 3 "~" H 6650 3450 50  0001 C CNN
@@
 L power:+12V #PWR0101
 U 1 1 5C4A87A7
-P 2400 900
-F 0 "#PWR0101" H 2400 750 50  0001 C CNN
-F 1 "+12V" H 2415 1073 50  0000 C CNN
-F 2 "" H 2400 900 50  0001 C CNN
-F 3 "" H 2400 900 50  0001 C CNN
-	1    2400 900
+P 9250 3000
+F 0 "#PWR0101" H 9250 2850 50  0001 C CNN
+F 1 "+12V" H 9265 3173 50  0000 C CNN
+F 2 "" H 9250 3000 50  0001 C CNN
+F 3 "" H 9250 3000 50  0001 C CNN
+	1    9250 3000
 	1    0    0    -1
 $EndComp
@@
 ADC_0_L1
 Wire Wire Line
-	2400 900  2400 950
+	9250 3000 9250 3050
 Wire Wire Line
 	2550 3550 2550 3500
@@
 L Connector:Screw_Terminal_01x02 J_in1
 U 1 1 5C4BF483
-P 1850 1250
-F 0 "J_in1" H 2050 1250 50  0000 C CNN
-F 1 "Screw_Terminal_01x02" H 2200 1000 50  0001 C CNN
-F 2 "TerminalBlock:TerminalBlock_Altech_AK300-2_P5.00mm" H 1850 1250 50  0001 C CNN
-F 3 "~" H 1850 1250 50  0001 C CNN
-	1    1850 1250
+P 8700 3350
+F 0 "J_in1" H 8900 3350 50  0000 C CNN
+F 1 "Screw_Terminal_01x02" H 9050 3100 50  0001 C CNN
+F 2 "TerminalBlock:TerminalBlock_Altech_AK300-2_P5.00mm" H 8700 3350 50  0001 C CNN
+F 3 "~" H 8700 3350 50  0001 C CNN
+	1    8700 3350
 	-1   0    0    1
 $EndComp
 Wire Wire Line
-	2050 1150 2050 950
+	8900 3250 8900 3050
 Wire Wire Line
 	2700 3250 2700 3300
@@
 L power:GND #PWR0102
 U 1 1 5C5456B4
-P 2050 1400
-F 0 "#PWR0102" H 2050 1150 50  0001 C CNN
-F 1 "GND" H 2055 1227 50  0000 C CNN
-F 2 "" H 2050 1400 50  0001 C CNN
-F 3 "" H 2050 1400 50  0001 C CNN
-	1    2050 1400
-	1    0    0    -1
-$EndComp
-Wire Wire Line
-	2050 950  2400 950
+P 8900 3500
+F 0 "#PWR0102" H 8900 3250 50  0001 C CNN
+F 1 "GND" H 8905 3327 50  0000 C CNN
+F 2 "" H 8900 3500 50  0001 C CNN
+F 3 "" H 8900 3500 50  0001 C CNN
+	1    8900 3500
+	1    0    0    -1
+$EndComp
+Wire Wire Line
+	8900 3050 9250 3050
 $Comp
 L oscila_mag-rescue:TC4420CPA-TC4420CPA-buck-rescue-buck_gnd-rescue-buck_vcc_sync-rescue U2
@@
 P 6650 4600
 F 0 "L2" V 6650 4815 50  0000 C CNN
-F 1 "50u" V 6500 4850 50  0000 C CNN
+F 1 "45.6u" V 6500 4850 50  0000 C CNN
 F 2 "Inductor_THT:L_Toroid_Horizontal_D12.7mm_P20.00mm_Diameter14-5mm_Amidon-T50" H 6650 4600 50  0001 C CNN
 F 3 "~" H 6650 4600 50  0001 C CNN
@@
 L Device:LED D9
 U 1 1 5D091513
-P 2400 1750
-F 0 "D9" V 2438 1633 50  0000 R CNN
-F 1 "LED" V 2347 1633 50  0000 R CNN
-F 2 "LED_THT:LED_D3.0mm_Clear" H 2400 1750 50  0001 C CNN
-F 3 "~" H 2400 1750 50  0001 C CNN
-	1    2400 1750
+P 9250 3850
+F 0 "D9" V 9288 3733 50  0000 R CNN
+F 1 "LED" V 9197 3733 50  0000 R CNN
+F 2 "LED_THT:LED_D3.0mm_Clear" H 9250 3850 50  0001 C CNN
+F 3 "~" H 9250 3850 50  0001 C CNN
+	1    9250 3850
 	0    -1   -1   0
 $EndComp
@@
 L Transistor_BJT:BC548 Q1
 U 1 1 5D091697
-P 2300 2250
-F 0 "Q1" H 2491 2296 50  0000 L CNN
-F 1 "BC548" H 2491 2205 50  0000 L CNN
-F 2 "Package_TO_SOT_THT:TO-92_Inline" H 2500 2175 50  0001 L CIN
-F 3 "http://www.fairchildsemi.com/ds/BC/BC547.pdf" H 2300 2250 50  0001 L CNN
-	1    2300 2250
+P 9150 4350
+F 0 "Q1" H 9341 4396 50  0000 L CNN
+F 1 "BC548" H 9341 4305 50  0000 L CNN
+F 2 "Package_TO_SOT_THT:TO-92_Inline" H 9350 4275 50  0001 L CIN
+F 3 "http://www.fairchildsemi.com/ds/BC/BC547.pdf" H 9150 4350 50  0001 L CNN
+	1    9150 4350
 	1    0    0    -1
 $EndComp
@@
 L Device:R R12
 U 1 1 5D09176F
-P 2400 1300
-F 0 "R12" H 2600 1300 50  0000 C CNN
-F 1 "560" H 2600 1200 50  0000 C CNN
-F 2 "Resistor_THT:R_Axial_DIN0207_L6.3mm_D2.5mm_P10.16mm_Horizontal" V 2330 1300 50  0001 C CNN
-F 3 "~" H 2400 1300 50  0001 C CNN
-	1    2400 1300
+P 9250 3400
+F 0 "R12" H 9450 3400 50  0000 C CNN
+F 1 "560" H 9450 3300 50  0000 C CNN
+F 2 "Resistor_THT:R_Axial_DIN0207_L6.3mm_D2.5mm_P10.16mm_Horizontal" V 9180 3400 50  0001 C CNN
+F 3 "~" H 9250 3400 50  0001 C CNN
+	1    9250 3400
 	1    0    0    -1
 $EndComp
@@
 L Device:R R10
 U 1 1 5D093C7C
-P 1800 2250
-F 0 "R10" V 2007 2250 50  0000 C CNN
-F 1 "50k" V 1916 2250 50  0000 C CNN
-F 2 "Resistor_THT:R_Axial_DIN0207_L6.3mm_D2.5mm_P10.16mm_Horizontal" V 1730 2250 50  0001 C CNN
-F 3 "~" H 1800 2250 50  0001 C CNN
-	1    1800 2250
+P 8650 4350
+F 0 "R10" V 8857 4350 50  0000 C CNN
+F 1 "50k" V 8766 4350 50  0000 C CNN
+F 2 "Resistor_THT:R_Axial_DIN0207_L6.3mm_D2.5mm_P10.16mm_Horizontal" V 8580 4350 50  0001 C CNN
+F 3 "~" H 8650 4350 50  0001 C CNN
+	1    8650 4350
 	0    -1   -1   0
 $EndComp
@@
 L power:GND #PWR07
 U 1 1 5D0ABD09
-P 2400 2600
-F 0 "#PWR07" H 2400 2350 50  0001 C CNN
-F 1 "GND" H 2405 2427 50  0000 C CNN
-F 2 "" H 2400 2600 50  0001 C CNN
-F 3 "" H 2400 2600 50  0001 C CNN
-	1    2400 2600
-	1    0    0    -1
-$EndComp
-Wire Wire Line
-	2400 1150 2400 950
-Connection ~ 2400 950
-Wire Wire Line
-	2050 1400 2050 1250
-Wire Wire Line
-	2400 1600 2400 1450
-Wire Wire Line
-	2400 1900 2400 2050
-Wire Wire Line
-	2400 2600 2400 2450
-Wire Wire Line
-	2100 2250 1950 2250
-Text GLabel 1350 2250 0    50   Input ~ 0
+P 9250 4700
+F 0 "#PWR07" H 9250 4450 50  0001 C CNN
+F 1 "GND" H 9255 4527 50  0000 C CNN
+F 2 "" H 9250 4700 50  0001 C CNN
+F 3 "" H 9250 4700 50  0001 C CNN
+	1    9250 4700
+	1    0    0    -1
+$EndComp
+Wire Wire Line
+	9250 3250 9250 3050
+Connection ~ 9250 3050
+Wire Wire Line
+	8900 3500 8900 3350
+Wire Wire Line
+	9250 3700 9250 3550
+Wire Wire Line
+	9250 4000 9250 4150
+Wire Wire Line
+	9250 4700 9250 4550
+Wire Wire Line
+	8950 4350 8800 4350
+Text GLabel 8200 4350 0    50   Input ~ 0
 DIGITAL_LED
 Wire Wire Line
-	1350 2250 1650 2250
+	8200 4350 8500 4350
 $Comp
 L pspice:CAP C6
