File: boost_311v/boost_311v.sch (KiCad schematic (older format))
At the start: 42 parts, among them Q1 BC556, Q2 PN2222A, Q3 2N3904, Q4 2N3906, Q5 IRFP260, Q6 2N3904, Q7 2N3906, U1 4N25, U4 LF357, U5 NE555

Commit message: Up pcb
Signed-off-by: fgl27 <fglfgl27@gmail.com>
Parts:
- removed Q3, Q6: 2N3904, Package_TO_SOT_THT:TO-92_Inline, symbol Transistor_BJT:2N3904
- removed Q4, Q7: 2N3906, Package_TO_SOT_THT:TO-92_Inline, symbol Transistor_BJT:2N3906
- removed U1: 4N25, Package_DIP:DIP-6_W7.62mm, symbol Isolator:4N25
- added C11: 10pF, Capacitor_THT:C_Disc_D7.5mm_W5.0mm_P5.00mm, symbol pspice:CAP
- added C12, C13, C14: 100pF, Capacitor_THT:C_Disc_D7.5mm_W5.0mm_P5.00mm, symbol pspice:CAP
- added J1: Vin, symbol Connector:Screw_Terminal_01x02
- added J2: VO, symbol Connector:Screw_Terminal_01x02
- added R11: 50kΩ, Resistor_THT:R_Axial_DIN0207_L6.3mm_D2.5mm_P10.16mm_Horizontal, symbol Device:R
- added R12: 10KΩ, Resistor_THT:R_Axial_DIN0207_L6.3mm_D2.5mm_P10.16mm_Horizontal, symbol Device:R
- added R13: 10kΩ, Resistor_THT:R_Axial_DIN0207_L6.3mm_D2.5mm_P10.16mm_Horizontal, symbol Device:R
- added U1: LM358, symbol Amplifier_Operational:LM358
- added U2: L7812, Package_TO_SOT_THT:TO-220-3_Vertical, symbol Regulator_Linear:LM7812_TO220
- added U3: TC4420CPA, DIP254P762X533-8, symbol 4420:TC4420CPA
- R3: value 1000kΩ -> 10MΩ
- R4: value 10kΩ -> 100kΩ
- R6: value 220Ω -> 220kΩ
- R7: value 470Ω -> 220kΩ
- R9: value 32kΩ -> 22kΩ
Connections:
- net +12V: no longer C10.1, C8.1, R14.1, R15.1, R2.2, R9.1, U4.7 (V+), U5.8 (VCC)
- net +24V: now also C13.1, J1.2 (Pin_2), U2.1 (VI)
- net GND: now also C13.2, C14.2, J1.1 (Pin_1), J2.2 (Pin_2), R13.2, U2.2 (GND), U3.4 (GND_2), U3.5 (GND); no longer R7.1
- net MOS_Gate: now also U3.6 (OUTPUT_2), U3.7 (OUTPUT)
- net PWM: no longer R6.2
- net at POT1.1: now also R7.2; no longer R9.2
- net at POT1.2: now also U1.5 (+); no longer U4.2 (-)
- net 12V_L7812: now reaches R6.1
- net 12V_L7812: now also C10.1, C8.1, R14.1, R15.1, R2.2, U4.7 (V+), U5.8 (VCC), C14.1, R12.1, U1.8 (V+), U2.3 (VO), U3.1 (VDD_2), U3.8 (VDD)
- net at D6.1 (K), R5.2: now also U3.2 (INPUT)
- net 1%VO_medição renamed 0,99%_VO
- net 0,99%_VO: now also R9.1
- net VO: no longer names the net of C9.1, D5.1 (K), R3.1
- net VO: now also J2.1 (Pin_1)
- new net: U1.1, U1.2 (-)
- new net: R12.2, R13.1, U1.3 (+)
- new net: C11.1, R11.1, R9.2, U1.6 (-)
- new net: C12.1, R11.2
- new net: R6.2, R7.1
- new net V_cnt: C11.2, C12.2, U1.7, U4.2 (-)
Other:
- note added: "1. Alimentação 15 a 30 V para 12 V"
- note added: "2. Onda dente de serra, F ≈ 46kHz"
- note added: "3. Comparador - Amplificação - PWM - duty 0 até 75%"
- note added: "4. Proteção PWM e acionamento MOSFET"
- note added: "5. Boost 24V para 311V - 0,3A"
- note added: "6. Controlador tipo II"
- note added: "7. LM358 Alimentação e proteção OP-AMP não usado"
- note added: "Ajustando o controle / potenciômetro\nAjusta a tensão de saída VO"
- note added: "O Duty é limitado em no máximo ≈ 75%\nImpedindo assim colocar a fonte em curto\n\nIsso ocorre pois a tensão máxima da dente de serra\né em torno de 7V, quando a tensão V_cnt > 7V a \nsaída do comparador vai para 0V\nO transistor amplifica e inverte a saída do comparador"
- note removed: "1. Geração dente de serra, F ≈ 46kHz"
- note removed: "2. Comparador - Amplificação - PWM - duty 0 até 73%"
- note removed: "3.1 Isolamento e acionamento MOSFET"
- note removed: "3.2 Isolamento e acionamento MOSFET"
- note removed: "4. Boost 24V para 311V - 0,3A"
- note removed: "Como o circuito foi desenvolvido para demostrar funcionamento de um boost\no Duty foi limitado a no máximo 73%, impedindo assim colocar a fonte em curto\n\nCaso a frequência necessária, impeça o uso do optocoupler, use o isolamento com diodo\nuse diodos com tensão reversa de pelo menos 100V"
- note removed: "O Duty é limitado em no máximo ≈ 73%\nImpedindo assim colocar a fonte em curto\nAjustável usando o Controle / potenciômetro"
- moved on the sheet: C1, C10, C2, C3, C4, C5, C6, C7, C8, C9, D1, D2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

Commit message: Up pcbs
Signed-off-by: fgl27 <fglfgl27@gmail.com>
Parts:
- added J3: Vin_boost, symbol Connector:Screw_Terminal_01x02
- J1: value Vin -> Vin_Cnt
Connections:
- net +24V: now also J3.2 (Pin_2)
- net GND: now also J3.1 (Pin_1)
Other:
- note added: "Ajustando o controle / potenciômetro\nAjusta-se a tensão de referência\ne assim ajusta-se a tensão de saída VO"
- note added: "Felipe Leon - 2021"
- note removed: "Ajustando o controle / potenciômetro\nAjusta a tensão de saída VO"
- moved on the sheet: C13, C14, D6, R12, R13, R5, U1A, U1C, U2, U3

Commit message: Up pcb
Signed-off-by: fgl27 <fglfgl27@gmail.com>
Parts:
- added POT2: 100kΩ, Potentiometer_THT:Potentiometer_Alps_RK163_Single_Horizontal, symbol Device:R_POT
- added R17: 1MΩ, Resistor_THT:R_Axial_DIN0207_L6.3mm_D2.5mm_P10.16mm_Horizontal, symbol Device:R
- added R18: 100kΩ, Resistor_THT:R_Axial_DIN0207_L6.3mm_D2.5mm_P10.16mm_Horizontal, symbol Device:R
- C1: value 2,2mF -> 100µF; footprint (none) -> Capacitor_THT:CP_Radial_D18.0mm_P7.50mm
- C5: value 100pF -> 500pF
- R3: value 10MΩ -> 1MΩ
- R4: value 100kΩ -> 10,1kΩ
Connections:
- net GND: now also R18.2
- net at C9.1, D5.1 (K), J2.1 (Pin_1)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: now also R17.1
- net 0,99%_VO renamed 1%_VO
- new net: POT2.3, R18.1
- new net 10%_VO: POT2.1, POT2.2, R17.2
Other:
- note added: "2. Onda dente de serra, F ≈ 13,33kHz"
- note removed: "2. Onda dente de serra, F ≈ 46kHz"
- moved on the sheet: R3, R4
Changed lines of the file:
@@
 $EndDescr
 Text Notes 6450 2450 0    79   ~ 0
-2. Onda dente de serra, F ≈ 46kHz
+2. Onda dente de serra, F ≈ 13,33kHz
 Text Notes 7000 1900 0    79   ~ 0
 Conversor CC-CC - Boost 24V para 311V - 0,3A
@@
 P 8100 4100
 F 0 "C5" H 8200 4250 50  0000 L CNN
-F 1 "100pF" H 8200 4000 50  0000 L CNN
+F 1 "500pF" H 8200 4000 50  0000 L CNN
 F 2 "Capacitor_THT:C_Disc_D7.5mm_W5.0mm_P5.00mm" H 8100 4100 50  0001 C CNN
 F 3 "~" H 8100 4100 50  0001 C CNN
@@
 $EndComp
 Text Label 11600 5550 2    59   ~ 0
-0,99%_VO
+1%_VO
 Wire Wire Line
 	11750 6750 11750 6650
@@
 	1    0    0    -1
 $EndComp
-Wire Wire Line
-	9400 6200 9950 6200
 $Comp
 L Connector:Screw_Terminal_01x02 J2
@@
 L Device:R R4
 U 1 1 614329D7
-P 9400 7350
-F 0 "R4" H 9550 7350 50  0000 C CNN
-F 1 "100kΩ" H 9600 7450 50  0000 C CNN
-F 2 "Resistor_THT:R_Axial_DIN0207_L6.3mm_D2.5mm_P10.16mm_Horizontal" V 9330 7350 50  0001 C CNN
-F 3 "~" H 9400 7350 50  0001 C CNN
-	1    9400 7350
+P 9850 7350
+F 0 "R4" H 10000 7350 50  0000 C CNN
+F 1 "10,1kΩ" H 10050 7450 50  0000 C CNN
+F 2 "Resistor_THT:R_Axial_DIN0207_L6.3mm_D2.5mm_P10.16mm_Horizontal" V 9780 7350 50  0001 C CNN
+F 3 "~" H 9850 7350 50  0001 C CNN
+	1    9850 7350
 	1    0    0    -1
 $EndComp
@@
 	-1   0    0    1
 $EndComp
-Text Notes 5650 7700 0    79   ~ 0
+Text Notes 5200 7750 0    79   ~ 0
 Tensão máxima, MOSFET, DIODOS e CAPACITORES 200V !!!
 Text Notes 9500 6050 0    49   ~ 0
@@
 5. Boost 24V para 311V - 0,3A
 Wire Wire Line
-	9400 7100 9500 7100
-Connection ~ 9400 7100
-Wire Wire Line
-	9400 7200 9400 7100
-Wire Wire Line
-	9400 7100 9400 6950
-Text Label 9500 7100 0    59   ~ 0
-0,99%_VO
+	9850 7050 9950 7050
+Connection ~ 9850 7050
+Wire Wire Line
+	9850 7050 9850 6950
+Text Label 9950 7050 0    59   ~ 0
+1%_VO
 Connection ~ 9400 6200
 Wire Wire Line
-	9400 6650 9400 6200
+	9850 6650 9850 6200
 $Comp
 L Device:R R3
 U 1 1 6143688B
-P 9400 6800
-F 0 "R3" H 9550 6800 50  0000 C CNN
-F 1 "10MΩ" H 9600 6900 50  0000 C CNN
-F 2 "Resistor_THT:R_Axial_DIN0207_L6.3mm_D2.5mm_P10.16mm_Horizontal" V 9330 6800 50  0001 C CNN
-F 3 "~" H 9400 6800 50  0001 C CNN
-	1    9400 6800
-	1    0    0    -1
-$EndComp
-Wire Wire Line
-	9400 7650 9400 7500
+P 9850 6800
+F 0 "R3" H 10000 6800 50  0000 C CNN
+F 1 "1MΩ" H 10050 6900 50  0000 C CNN
+F 2 "Resistor_THT:R_Axial_DIN0207_L6.3mm_D2.5mm_P10.16mm_Horizontal" V 9780 6800 50  0001 C CNN
+F 3 "~" H 9850 6800 50  0001 C CNN
+	1    9850 6800
+	1    0    0    -1
+$EndComp
+Wire Wire Line
+	9850 7650 9850 7500
 $Comp
 L power:GND #PWR017
 U 1 1 614329DD
-P 9400 7650
-F 0 "#PWR017" H 9400 7400 50  0001 C CNN
-F 1 "GND" H 9405 7477 50  0000 C CNN
-F 2 "" H 9400 7650 50  0001 C CNN
-F 3 "" H 9400 7650 50  0001 C CNN
-	1    9400 7650
+P 9850 7650
+F 0 "#PWR017" H 9850 7400 50  0001 C CNN
+F 1 "GND" H 9855 7477 50  0000 C CNN
+F 2 "" H 9850 7650 50  0001 C CNN
+F 3 "" H 9850 7650 50  0001 C CNN
+	1    9850 7650
 	1    0    0    -1
 $EndComp
@@
 Wire Wire Line
 	9400 6200 9400 5900
-Wire Wire Line
-	9150 6200 9400 6200
 $Comp
 L Device:CP C7
@@
 P 5800 6800
 F 0 "C1" H 5600 6800 50  0000 L CNN
-F 1 "2,2mF" H 5550 6700 50  0000 L CNN
-F 2 "" H 5838 6650 50  0001 C CNN
+F 1 "100µF" H 5550 6700 50  0000 L CNN
+F 2 "Capacitor_THT:CP_Radial_D18.0mm_P7.50mm" H 5838 6650 50  0001 C CNN
 F 3 "~" H 5800 6800 50  0001 C CNN
 	1    5800 6800
@@
 Text Notes 11350 9500 0    79   ~ 0
 Felipe Leon - 2021
+$Comp
+L Device:R R18
+U 1 1 613AAFEF
+P 9200 7350
+F 0 "R18" H 9350 7300 50  0000 C CNN
+F 1 "100kΩ" H 9400 7400 50  0000 C CNN
+F 2 "Resistor_THT:R_Axial_DIN0207_L6.3mm_D2.5mm_P10.16mm_Horizontal" V 9130 7350 50  0001 C CNN
+F 3 "~" H 9200 7350 50  0001 C CNN
+	1    9200 7350
+	1    0    0    -1
+$EndComp
+Wire Wire Line
+	9200 6900 9200 6850
+Text Label 9450 7050 0    59   ~ 0
+10%_VO
+$Comp
+L Device:R R17
+U 1 1 613AAFFB
+P 9200 6650
+F 0 "R17" H 9350 6600 50  0000 C CNN
+F 1 "1MΩ" H 9350 6700 50  0000 C CNN
+F 2 "Resistor_THT:R_Axial_DIN0207_L6.3mm_D2.5mm_P10.16mm_Horizontal" V 9130 6650 50  0001 C CNN
+F 3 "~" H 9200 6650 50  0001 C CNN
+	1    9200 6650
+	1    0    0    -1
+$EndComp
+Wire Wire Line
+	9200 7650 9200 7500
+$Comp
+L power:GND #PWR02
+U 1 1 613AB002
+P 9200 7650
+F 0 "#PWR02" H 9200 7400 50  0001 C CNN
+F 1 "GND" H 9205 7477 50  0000 C CNN
+F 2 "" H 9200 7650 50  0001 C CNN
+F 3 "" H 9200 7650 50  0001 C CNN
+	1    9200 7650
+	1    0    0    -1
+$EndComp
+$Comp
+L Device:R_POT POT2
+U 1 1 613DE305
+P 9200 7050
+F 0 "POT2" H 9100 7100 50  0000 R CNN
+F 1 "100kΩ" H 9150 7000 50  0000 R CNN
+F 2 "Potentiometer_THT:Potentiometer_Alps_RK163_Single_Horizontal" H 9200 7050 50  0001 C CNN
+F 3 "~" H 9200 7050 50  0001 C CNN
+	1    9200 7050
+	1    0    0    -1
+$EndComp
+Wire Wire Line
+	9150 6200 9200 6200
+Wire Wire Line
+	9200 6500 9200 6200
+Connection ~ 9200 6200
+Wire Wire Line
+	9200 6200 9400 6200
+Connection ~ 9850 6200
+Wire Wire Line
+	9850 6200 9950 6200
+Wire Wire Line
+	9400 6200 9850 6200
+Wire Wire Line
+	9450 7050 9350 7050
+Wire Wire Line
+	9350 7050 9350 6850
+Wire Wire Line
+	9350 6850 9200 6850
+Connection ~ 9350 7050
+Connection ~ 9200 6850
+Wire Wire Line
+	9200 6850 9200 6800
+Wire Wire Line
+	9850 7050 9850 7200
 $EndSCHEMATC

Commit message: Up pcb
Signed-off-by: fgl27 <fglfgl27@gmail.com>
Parts:
- added C15: 100nF, Capacitor_THT:C_Disc_D7.5mm_W5.0mm_P5.00mm, symbol pspice:CAP
- added D7: D_Zener_6,5V, symbol Device:D_Zener
- added R19: 1kΩ, Resistor_THT:R_Axial_DIN0207_L6.3mm_D2.5mm_P10.16mm_Horizontal, symbol Device:R
- C13: value 100pF -> 10µF
- C14: value 100pF -> 100nF
Connections:
- net 12V_L7812: now also C15.1
- net GND: now also U1.4 (V-), C15.2, D7.1 (K)
- net V_cnt: now also R19.1; no longer U4.2 (-)
- net V_REF: now reaches POT1.2, U1.5 (+)
- new net: D7.2 (A), R19.2, U4.2 (-)
Other:
- note added: "3. Comparador - Amplificação - PWM - duty 0 até 73%"
- note added: "O Duty é limitado em no máximo ≈ 73%\nImpedindo assim colocar a fonte em curto\n\nTensão dente de serra é em torno de 8.8V, zener 6,5V\n\nO transistor amplifica e inverte a saída do comparador"
- note removed: "3. Comparador - Amplificação - PWM - duty 0 até 75%"
- note removed: "O Duty é limitado em no máximo ≈ 75%\nImpedindo assim colocar a fonte em curto\n\nIsso ocorre pois a tensão máxima da dente de serra\né em torno de 7V, quando a tensão V_cnt > 7V a \nsaída do comparador vai para 0V\nO transistor amplifica e inverte a saída do comparador"
- moved on the sheet: R12, R13, U1A, U1C
Changed lines of the file:
@@
 Conversor CC-CC - Boost 24V para 311V - 0,3A
 Text Notes 10650 2400 0    79   ~ 0
-3. Comparador - Amplificação - PWM - duty 0 até 75%
+3. Comparador - Amplificação - PWM - duty 0 até 73%
 Wire Notes Line
 	5500 4600 5500 2550
@@
 Wire Wire Line
 	12200 3200 12200 2900
-Text Notes 11000 4650 0    59   ~ 0
-O Duty é limitado em no máximo ≈ 75%\nImpedindo assim colocar a fonte em curto\n\nIsso ocorre pois a tensão máxima da dente de serra\né em torno de 7V, quando a tensão V_cnt > 7V a \nsaída do comparador vai para 0V\nO transistor amplifica e inverte a saída do comparador
-Text Label 12000 3600 2    59   ~ 0
+Text Notes 11100 4700 0    59   ~ 0
+O Duty é limitado em no máximo ≈ 73%\nImpedindo assim colocar a fonte em curto\n\nTensão dente de serra é em torno de 8.8V, zener 6,5V\n\nO transistor amplifica e inverte a saída do comparador
+Text Label 11350 3600 2    59   ~ 0
 V_cnt
 $Comp
@@
 P 4200 3200
 F 0 "C14" H 4300 3350 50  0000 L CNN
-F 1 "100pF" H 4300 3100 50  0000 L CNN
+F 1 "100nF" H 4300 3100 50  0000 L CNN
 F 2 "Capacitor_THT:C_Disc_D7.5mm_W5.0mm_P5.00mm" H 4200 3200 50  0001 C CNN
 F 3 "~" H 4200 3200 50  0001 C CNN
@@
 P 3050 3200
 F 0 "C13" H 3150 3350 50  0000 L CNN
-F 1 "100pF" H 3150 3100 50  0000 L CNN
+F 1 "10µF" H 3150 3100 50  0000 L CNN
 F 2 "Capacitor_THT:C_Disc_D7.5mm_W5.0mm_P5.00mm" H 3050 3200 50  0001 C CNN
 F 3 "~" H 3050 3200 50  0001 C CNN
@@
 Text Notes 11300 7250 0    59   ~ 0
 Ajustando o controle / potenciômetro\nAjusta-se a tensão de referência\ne assim ajusta-se a tensão de saída VO
-Wire Wire Line
-	11000 6750 11000 6150
-Text Label 11000 6750 0    59   ~ 0
+Text Label 11000 5950 0    59   ~ 0
 12V_L7812
 Wire Notes Line
@@
 	1    0    0    -1
 $EndComp
-Wire Notes Line
-	10850 7700 10850 9000
-Wire Notes Line
-	13100 9000 10850 9000
-Wire Notes Line
-	13100 7700 13100 9000
-Wire Notes Line
-	10850 7700 13100 7700
 Text Notes 10700 7550 0    79   ~ 0
 7. LM358 Alimentação e proteção OP-AMP não usado
 Wire Wire Line
-	12850 8650 12850 8400
-Wire Wire Line
-	12250 8650 12850 8650
-Wire Wire Line
-	12250 8500 12250 8650
-Connection ~ 11850 8300
-Wire Wire Line
-	12250 8300 11850 8300
-Wire Wire Line
-	11850 7900 11200 7900
-Wire Wire Line
-	11850 8000 11850 7900
+	13550 8700 13550 8450
+Wire Wire Line
+	12950 8700 13550 8700
+Wire Wire Line
+	12950 8550 12950 8700
+Connection ~ 12550 8350
+Wire Wire Line
+	12950 8350 12550 8350
+Wire Wire Line
+	12550 7950 11900 7950
+Wire Wire Line
+	12550 8050 12550 7950
 $Comp
 L Device:R R13
 U 1 1 6176F609
-P 11850 8450
-F 0 "R13" H 12000 8450 50  0000 C CNN
-F 1 "10kΩ" H 12050 8550 50  0000 C CNN
-F 2 "Resistor_THT:R_Axial_DIN0207_L6.3mm_D2.5mm_P10.16mm_Horizontal" V 11780 8450 50  0001 C CNN
-F 3 "~" H 11850 8450 50  0001 C CNN
-	1    11850 8450
+P 12550 8500
+F 0 "R13" H 12700 8500 50  0000 C CNN
+F 1 "10kΩ" H 12750 8600 50  0000 C CNN
+F 2 "Resistor_THT:R_Axial_DIN0207_L6.3mm_D2.5mm_P10.16mm_Horizontal" V 12480 8500 50  0001 C CNN
+F 3 "~" H 12550 8500 50  0001 C CNN
+	1    12550 8500
 	1    0    0    -1
 $EndComp
@@
 L Device:R R12
 U 1 1 6176F5FC
-P 11850 8150
-F 0 "R12" H 12000 8150 50  0000 C CNN
-F 1 "10KΩ" H 12050 8250 50  0000 C CNN
-F 2 "Resistor_THT:R_Axial_DIN0207_L6.3mm_D2.5mm_P10.16mm_Horizontal" V 11780 8150 50  0001 C CNN
-F 3 "~" H 11850 8150 50  0001 C CNN
-	1    11850 8150
+P 12550 8200
+F 0 "R12" H 12700 8200 50  0000 C CNN
+F 1 "10KΩ" H 12750 8300 50  0000 C CNN
+F 2 "Resistor_THT:R_Axial_DIN0207_L6.3mm_D2.5mm_P10.16mm_Horizontal" V 12480 8200 50  0001 C CNN
+F 3 "~" H 12550 8200 50  0001 C CNN
+	1    12550 8200
 	1    0    0    -1
 $EndComp
@@
 L power:GND #PWR025
 U 1 1 6176F5F5
-P 11850 8600
-F 0 "#PWR025" H 11850 8350 50  0001 C CNN
-F 1 "GND" H 11855 8427 50  0000 C CNN
-F 2 "" H 11850 8600 50  0001 C CNN
-F 3 "" H 11850 8600 50  0001 C CNN
-	1    11850 8600
+P 12550 8650
+F 0 "#PWR025" H 12550 8400 50  0001 C CNN
+F 1 "GND" H 12555 8477 50  0000 C CNN
+F 2 "" H 12550 8650 50  0001 C CNN
+F 3 "" H 12550 8650 50  0001 C CNN
+	1    12550 8650
 	1    0    0    -1
 $EndComp
@@
 L power:GND #PWR024
 U 1 1 61740376
-P 11200 8600
-F 0 "#PWR024" H 11200 8350 50  0001 C CNN
-F 1 "GND" H 11205 8427 50  0000 C CNN
-F 2 "" H 11200 8600 50  0001 C CNN
-F 3 "" H 11200 8600 50  0001 C CNN
-	1    11200 8600
-	1    0    0    -1
-$EndComp
-Text Label 11200 7900 0    59   ~ 0
+P 11900 8650
+F 0 "#PWR024" H 11900 8400 50  0001 C CNN
+F 1 "GND" H 11905 8477 50  0000 C CNN
+F 2 "" H 11900 8650 50  0001 C CNN
+F 3 "" H 11900 8650 50  0001 C CNN
+	1    11900 8650
+	1    0    0    -1
+$EndComp
+Text Label 11450 7950 2    59   ~ 0
 12V_L7812
 $Comp
 L Amplifier_Operational:LM358 U1
 U 3 1 613DEC29
-P 11300 8200
-F 0 "U1" H 11258 8246 50  0000 L CNN
-F 1 "LM358" H 11258 8155 50  0000 L CNN
-F 2 "" H 11300 8200 50  0001 C CNN
-F 3 "http://www.ti.com/lit/ds/symlink/lm2904-n.pdf" H 11300 8200 50  0001 C CNN
-	3    11300 8200
+P 12000 8250
+F 0 "U1" H 11958 8296 50  0000 L CNN
+F 1 "LM358" H 11958 8205 50  0000 L CNN
+F 2 "" H 12000 8250 50  0001 C CNN
+F 3 "http://www.ti.com/lit/ds/symlink/lm2904-n.pdf" H 12000 8250 50  0001 C CNN
+	3    12000 8250
 	1    0    0    -1
 $EndComp
@@
 L Amplifier_Operational:LM358 U1
 U 1 1 613DA37F
-P 12550 8400
-F 0 "U1" H 12550 8767 50  0000 C CNN
-F 1 "LM358" H 12550 8676 50  0000 C CNN
-F 2 "" H 12550 8400 50  0001 C CNN
-F 3 "http://www.ti.com/lit/ds/symlink/lm2904-n.pdf" H 12550 8400 50  0001 C CNN
-	1    12550 8400
+P 13250 8450
+F 0 "U1" H 13250 8817 50  0000 C CNN
+F 1 "LM358" H 13250 8726 50  0000 C CNN
+F 2 "" H 13250 8450 50  0001 C CNN
+F 3 "http://www.ti.com/lit/ds/symlink/lm2904-n.pdf" H 13250 8450 50  0001 C CNN
+	1    13250 8450
 	1    0    0    -1
 $EndComp
@@
 Wire Wire Line
 	9850 7050 9850 7200
+$Comp
+L Device:D_Zener D7
+U 1 1 6138527C
+P 11800 3750
+F 0 "D7" V 11800 3950 50  0000 R CNN
+F 1 "D_Zener_6,5V" V 11700 4300 50  0000 R CNN
+F 2 "" H 11800 3750 50  0001 C CNN
+F 3 "~" H 11800 3750 50  0001 C CNN
+	1    11800 3750
+	0    -1   -1   0
+$EndComp
+$Comp
+L power:GND #PWR06
+U 1 1 61393844
+P 11800 3900
+F 0 "#PWR06" H 11800 3650 50  0001 C CNN
+F 1 "GND" H 11805 3727 50  0000 C CNN
+F 2 "" H 11800 3900 50  0001 C CNN
+F 3 "" H 11800 3900 50  0001 C CNN
+	1    11800 3900
+	1    0    0    -1
+$EndComp
+Wire Wire Line
+	11800 3600 11650 3600
+$Comp
+L Device:R R19
+U 1 1 613A866C
+P 11500 3600
+F 0 "R19" V 11700 3600 50  0000 C CNN
+F 1 "1kΩ" V 11600 3600 50  0000 C CNN
+F 2 "Resistor_THT:R_Axial_DIN0207_L6.3mm_D2.5mm_P10.16mm_Horizontal" V 11430 3600 50  0001 C CNN
+F 3 "~" H 11500 3600 50  0001 C CNN
+	1    11500 3600
+	0    -1   -1   0
+$EndComp
+Wire Wire Line
+	11800 3600 12000 3600
+Connection ~ 11800 3600
+$Comp
+L pspice:CAP C15
+U 1 1 613D8A3F
+P 11550 8400
+F 0 "C15" H 11200 8550 50  0000 L CNN
+F 1 "100nF" H 11150 8250 50  0000 L CNN
+F 2 "Capacitor_THT:C_Disc_D7.5mm_W5.0mm_P5.00mm" H 11550 8400 50  0001 C CNN
+F 3 "~" H 11550 8400 50  0001 C CNN
+	1    11550 8400
+	1    0    0    -1
+$EndComp
+$Comp
+L power:GND #PWR07
+U 1 1 613D8A45
+P 11550 8650
+F 0 "#PWR07" H 11550 8400 50  0001 C CNN
+F 1 "GND" H 11555 8477 50  0000 C CNN
+F 2 "" H 11550 8650 50  0001 C CNN
+F 3 "" H 11550 8650 50  0001 C CNN
+	1    11550 8650
+	1    0    0    -1
+$EndComp
+Wire Wire Line
+	11550 8150 11550 7950
+Wire Wire Line
+	11550 7950 11900 7950
+Connection ~ 11900 7950
+Wire Wire Line
+	11900 8650 11900 8550
+Wire Wire Line
+	11550 7950 11450 7950
+Connection ~ 11550 7950
+Wire Notes Line
+	13750 7700 13750 9050
+Wire Notes Line
+	10850 7700 13750 7700
+Wire Notes Line
+	10850 7700 10850 9050
+Wire Notes Line
+	10850 9050 13750 9050
+Wire Wire Line
+	11000 6150 11000 5950
+Text Label 12050 6500 0    50   ~ 0
+V_REF
 $EndSCHEMATC

Commit message: Up pcb
Signed-off-by: fgl27 <fglfgl27@gmail.com>
Parts:
- removed POT2: 100kΩ, Potentiometer_THT:Potentiometer_Alps_RK163_Single_Horizontal, symbol Device:R_POT
- added C16: 10nF, Capacitor_THT:C_Disc_D7.5mm_W5.0mm_P5.00mm, symbol pspice:CAP
- added TRIM_POT1: 22kΩ, symbol Device:R_POT_TRIM
- added TRIM_POT2: 100kΩ, symbol Device:R_POT_TRIM
- D7: value D_Zener_6,5V -> Zener 6,5V
- R14: value 10kΩ -> 1kΩ
- R8: value 470Ω -> 330Ω
Connections:
- net +12V is gone; now on net 12V_L7812: U5.4 (R)
- net 10%_VO: now also TRIM_POT2.1, TRIM_POT2.2
- net 12V_L7812: now also C10.2, C16.1; no longer C10.1
- net GND: now also C10.1, C16.2; no longer C10.2
- net at R14.2: now also TRIM_POT1.1, TRIM_POT1.2; no longer Q1.3 (E)
- net at R18.1: now also TRIM_POT2.3
- new net: Q1.3 (E), TRIM_POT1.3
Other:
- note added: "2. Onda dente de serra, F ≈ 5,5 até 100 kHz"
- note added: "3. Comparador - Amplificação - PWM - duty 0 até 75%"
- note added: "O Duty é limitado em no máximo ≈ 75%\nImpedindo assim colocar a fonte em curto\n\nTensão dente de serra é em torno de 8.8V, zener 6,5V\n\nO transistor amplifica e inverte a saída do comparador"
- note removed: "2. Onda dente de serra, F ≈ 13,33kHz"
- note removed: "3. Comparador - Amplificação - PWM - duty 0 até 73%"
- note removed: "O Duty é limitado em no máximo ≈ 73%\nImpedindo assim colocar a fonte em curto\n\nTensão dente de serra é em torno de 8.8V, zener 6,5V\n\nO transistor amplifica e inverte a saída do comparador"
- moved on the sheet: C10, Q1, R14, R15, R16

Commit message: Up ocb
Signed-off-by: fgl27 <fglfgl27@gmail.com>
Other:
- note added: "Ajustando o trimpot se a ajusta a frequência de operação"
- moved on the sheet: C4, C5, C8, Q1, R14, R15, R16, R8, TRIM_POT1, U5

Commit message: Up pcb
Signed-off-by: fgl27 <fglfgl27@gmail.com>
Parts:
- removed R17: 1MΩ, Resistor_THT:R_Axial_DIN0207_L6.3mm_D2.5mm_P10.16mm_Horizontal, symbol Device:R
- added R20, R21, R23, R24: 330kΩ, Resistor_THT:R_Axial_DIN0207_L6.3mm_D2.5mm_P10.16mm_Horizontal, symbol Device:R
- added R22: 220kΩ, Resistor_THT:R_Axial_DIN0207_L6.3mm_D2.5mm_P10.16mm_Horizontal, symbol Device:R
- R3: value 1MΩ -> 330kΩ
- R4: value 10,1kΩ -> 10kΩ
- TRIM_POT2: value 100kΩ -> 22kΩ
Connections:
- net 10%_VO: now also R22.2
- net at C9.1, D5.1 (K), J2.1 (Pin_1): now also R20.1, R23.1; no longer R3.1
- new net: R23.2, R24.1
- new net: R24.2, R3.1
- new net: R21.2, R22.1
- new net: R20.2, R21.1
Other:
- note added: "10% VO ponto de medição com osciloscópio\nProbe osciloscópio em 10X e osciloscópio em 100X"
- note added: "Tensão máxima\nMOSFET, DIODOS, CAPACITORES e RESISTORES de 1/4 é 200V !!!"
- note removed: "Tensão máxima, MOSFET, DIODOS e CAPACITORES 200V !!!"
- moved on the sheet: R18, R3, R4, TRIM_POT2
