File: boost_311v/boost_311v.sch (KiCad schematic (older format))
At the start: 58 parts, among them J2 VO, J3 Vin_boost, Q1 BC556, Q2 PN2222A, Q3 PN2222A, Q4 PN2222A, Q5 IRFP260, Q6 2N3904, Q7 2N3906, U2 L7812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

Commit message: Up pcb
Signed-off-by: fgl27 <fglfgl27@gmail.com>
Other:
- note added: "Tensão máxima\nMOSFET, DIODOS, CAPACITORES e RESISTORES de 1/4 é 200V !!!\n\nCorrente de média Mosfet ≈ 5A\nCorrente de pico Mosfet ≈ 25A\n\nCorrente de média Diodos = Io ≈ 0,3A se Ro = 1kΩ\nCorrente de pico Diodos ≈ 14A"
- note removed: "Tensão máxima\nMOSFET, DIODOS, CAPACITORES e RESISTORES de 1/4 é 200V !!!\nCOrrente de pico Mosfet ≈ 5A"
Changed lines of the file:
@@
 	0    -1   -1   0
 $EndComp
-Text Notes 9100 6950 0    79   ~ 0
-                   Tensão máxima\nMOSFET, DIODOS, CAPACITORES e RESISTORES de 1/4 é 200V !!!\nCOrrente de pico Mosfet ≈ 5A
+Text Notes 8900 7450 0    69   ~ 0
+                   Tensão máxima\nMOSFET, DIODOS, CAPACITORES e RESISTORES de 1/4 é 200V !!!\n\nCorrente de média Mosfet ≈ 5A\nCorrente de pico   Mosfet ≈ 25A\n\nCorrente de média Diodos = Io ≈ 0,3A se Ro = 1kΩ\nCorrente de pico   Diodos ≈ 14A
 Text Notes 13950 5150 0    49   ~ 0
 Carga Máxima 0,3A\n1kΩ quando VO = 311V
@@
 Wire Notes Line
 	8700 4350 8700 7800
-Text Notes 10750 7650 0    79   ~ 0
+Text Notes 11150 7700 0    69   ~ 0
 10% VO ponto de medição com osciloscópio\nProbe osciloscópio em 10X e osciloscópio em 100X\nAjustando o trimpot  para obter perfeito 10%
 $Comp

Commit message: Up pcb
Signed-off-by: fgl27 <fglfgl27@gmail.com>
Other:
- note added: "Tensão máxima\nMOSFET, DIODOS, CAPACITORES e RESISTORES de 1/4 é 200V !!!\n\nCorrente média Mosfet ≈ 5A\nCorrente de pico Mosfet ≈ 25A\n\nCorrente média Diodos = Io ≈ 0,3A se Ro = 1kΩ\nCorrente de pico Diodos ≈ 14A"
- note removed: "Tensão máxima\nMOSFET, DIODOS, CAPACITORES e RESISTORES de 1/4 é 200V !!!\n\nCorrente de média Mosfet ≈ 5A\nCorrente de pico Mosfet ≈ 25A\n\nCorrente de média Diodos = Io ≈ 0,3A se Ro = 1kΩ\nCorrente de pico Diodos ≈ 14A"
Changed lines of the file:
@@
 $EndComp
 Text Notes 8900 7450 0    69   ~ 0
-                   Tensão máxima\nMOSFET, DIODOS, CAPACITORES e RESISTORES de 1/4 é 200V !!!\n\nCorrente de média Mosfet ≈ 5A\nCorrente de pico   Mosfet ≈ 25A\n\nCorrente de média Diodos = Io ≈ 0,3A se Ro = 1kΩ\nCorrente de pico   Diodos ≈ 14A
+                   Tensão máxima\nMOSFET, DIODOS, CAPACITORES e RESISTORES de 1/4 é 200V !!!\n\nCorrente média   Mosfet ≈ 5A\nCorrente de pico Mosfet ≈ 25A\n\nCorrente média   Diodos = Io ≈ 0,3A se Ro = 1kΩ\nCorrente de pico Diodos ≈ 14A
 Text Notes 13950 5150 0    49   ~ 0
 Carga Máxima 0,3A\n1kΩ quando VO = 311V

Commit message: Up pcb
Signed-off-by: fgl27 <fglfgl27@gmail.com>
Parts:
- added J1: Vin_cnt, TerminalBlock:TerminalBlock_Altech_AK300-2_P5.00mm, symbol Connector:Screw_Terminal_01x02
- C1: footprint Capacitor_THT:CP_Radial_D18.0mm_P7.50mm -> Capacitor_THT:CP_Radial_D12.5mm_P5.00mm
- C11, C2, C3, C7, C9: footprint Capacitor_THT:CP_Radial_D18.0mm_P7.50mm -> Capacitor_THT:CP_Radial_D16.0mm_P7.50mm
- C12, C15: footprint Capacitor_THT:CP_Radial_D18.0mm_P7.50mm -> Capacitor_THT:CP_Radial_D22.0mm_P10.00mm_SnapIn
- HS1: footprint (none) -> Heatsink:Heatsink_Stonecold_HS-132_32x14mm_2xFixation1.5mm
- J2, J3: footprint (none) -> TerminalBlock:TerminalBlock_Altech_AK300-2_P5.00mm
- L1: footprint (none) -> Inductor_THT:L_Toroid_Vertical_L21.6mm_W9.1mm_P8.40mm_Bourns_5700
- Q2, Q3, Q4, Q6, Q7: footprint Package_TO_SOT_THT:TO-92_Inline -> Package_TO_SOT_THT:TO-92_Wide
- TRIM_POT1, TRIM_POT2: footprint (none) -> Potentiometer_THT:Potentiometer_ACP_CA6-H2,5_Horizontal
- renumbered D6 to D5
Connections:
- net +12V: now also J1.2 (Pin_2)
- net GND1: now also J1.1 (Pin_1)
Changed lines of the file:
@@
 F 0 "Q2" H 11390 2546 50  0000 L CNN
 F 1 "PN2222A" H 11390 2455 50  0000 L CNN
-F 2 "Package_TO_SOT_THT:TO-92_Inline" H 11400 2425 50  0001 L CIN
+F 2 "Package_TO_SOT_THT:TO-92_Wide" H 11400 2425 50  0001 L CIN
 F 3 "https://www.onsemi.com/pub/Collateral/PN2222-D.PDF" H 11200 2500 50  0001 L CNN
 	1    11200 2500
@@
 F 0 "J2" H 14600 5250 50  0001 C CNN
 F 1 "VO" H 14600 5250 50  0000 C CNN
-F 2 "" H 14450 5300 50  0001 C CNN
+F 2 "TerminalBlock:TerminalBlock_Altech_AK300-2_P5.00mm" H 14450 5300 50  0001 C CNN
 F 3 "~" H 14450 5300 50  0001 C CNN
 	1    14450 5300
@@
 F 0 "C3" V 12150 5250 50  0000 L CNN
 F 1 "100µF_200V" V 12250 5050 50  0000 L CNN
-F 2 "Capacitor_THT:CP_Radial_D18.0mm_P7.50mm" H 12038 5150 50  0001 C CNN
+F 2 "Capacitor_THT:CP_Radial_D16.0mm_P7.50mm" H 12038 5150 50  0001 C CNN
 F 3 "~" H 12000 5300 50  0001 C CNN
 	1    12000 5300
@@
 F 0 "C2" H 11668 6146 50  0000 L CNN
 F 1 "100µF" H 11668 6055 50  0000 L CNN
-F 2 "Capacitor_THT:CP_Radial_D18.0mm_P7.50mm" H 11588 5950 50  0001 C CNN
+F 2 "Capacitor_THT:CP_Radial_D16.0mm_P7.50mm" H 11588 5950 50  0001 C CNN
 F 3 "~" H 11550 6100 50  0001 C CNN
 	1    11550 6100
@@
 F 0 "HS1" H 10842 6671 50  0000 L CNN
 F 1 "Heatsink" H 10842 6580 50  0000 L CNN
-F 2 "" H 10712 6550 50  0001 C CNN
+F 2 "Heatsink:Heatsink_Stonecold_HS-132_32x14mm_2xFixation1.5mm" H 10712 6550 50  0001 C CNN
 F 3 "~" H 10712 6550 50  0001 C CNN
 	1    10700 6550
@@
 F 0 "L1" H 10150 5965 50  0000 C CNN
 F 1 "20µH" H 10150 5874 50  0000 C CNN
-F 2 "" H 10150 5750 50  0001 C CNN
+F 2 "Inductor_THT:L_Toroid_Vertical_L21.6mm_W9.1mm_P8.40mm_Bourns_5700" H 10150 5750 50  0001 C CNN
 F 3 "~" H 10150 5750 50  0001 C CNN
 	1    10150 5750
@@
 F 0 "C1" H 9250 6100 50  0000 L CNN
 F 1 "100µF" H 9150 6000 50  0000 L CNN
-F 2 "Capacitor_THT:CP_Radial_D18.0mm_P7.50mm" H 9538 5900 50  0001 C CNN
+F 2 "Capacitor_THT:CP_Radial_D12.5mm_P5.00mm" H 9538 5900 50  0001 C CNN
 F 3 "~" H 9500 6050 50  0001 C CNN
 	1    9500 6050
@@
 F 0 "J3" H 8900 5950 50  0001 C CNN
 F 1 "Vin_boost" H 8900 5900 50  0000 C CNN
-F 2 "" H 8900 6150 50  0001 C CNN
+F 2 "TerminalBlock:TerminalBlock_Altech_AK300-2_P5.00mm" H 8900 6150 50  0001 C CNN
 F 3 "~" H 8900 6150 50  0001 C CNN
 	1    8900 6150
@@
 F 0 "TRIM_POT1" H 7280 2296 50  0000 R CNN
 F 1 "22kΩ" H 7280 2205 50  0000 R CNN
-F 2 "" H 7350 2250 50  0001 C CNN
+F 2 "Potentiometer_THT:Potentiometer_ACP_CA6-H2,5_Horizontal" H 7350 2250 50  0001 C CNN
 F 3 "~" H 7350 2250 50  0001 C CNN
 	1    7350 2250
@@
 F 0 "TRIM_POT2" H 13980 6896 50  0000 R CNN
 F 1 "22kΩ" H 13980 6805 50  0000 R CNN
-F 2 "" H 14050 6850 50  0001 C CNN
+F 2 "Potentiometer_THT:Potentiometer_ACP_CA6-H2,5_Horizontal" H 14050 6850 50  0001 C CNN
 F 3 "~" H 14050 6850 50  0001 C CNN
 	1    14050 6850
@@
 F 0 "Q3" H 3590 6446 50  0000 L CNN
 F 1 "PN2222A" H 3590 6355 50  0000 L CNN
-F 2 "Package_TO_SOT_THT:TO-92_Inline" H 3600 6325 50  0001 L CIN
+F 2 "Package_TO_SOT_THT:TO-92_Wide" H 3600 6325 50  0001 L CIN
 F 3 "https://www.onsemi.com/pub/Collateral/PN2222-D.PDF" H 3400 6400 50  0001 L CNN
 	1    3400 6400
@@
 F 0 "Q4" H 4240 6246 50  0000 L CNN
 F 1 "PN2222A" H 4240 6155 50  0000 L CNN
-F 2 "Package_TO_SOT_THT:TO-92_Inline" H 4250 6125 50  0001 L CIN
+F 2 "Package_TO_SOT_THT:TO-92_Wide" H 4250 6125 50  0001 L CIN
 F 3 "https://www.onsemi.com/pub/Collateral/PN2222-D.PDF" H 4050 6200 50  0001 L CNN
 	1    4050 6200
@@
 F 0 "Q7" H 5140 6446 50  0000 L CNN
 F 1 "2N3906" H 5140 6355 50  0000 L CNN
-F 2 "Package_TO_SOT_THT:TO-92_Inline" H 5150 6325 50  0001 L CIN
+F 2 "Package_TO_SOT_THT:TO-92_Wide" H 5150 6325 50  0001 L CIN
 F 3 "https://www.onsemi.com/pub/Collateral/2N3906-D.PDF" H 4950 6400 50  0001 L CNN
 	1    4950 6400
@@
 F 0 "Q6" H 5140 6046 50  0000 L CNN
 F 1 "2N3904" H 5140 5955 50  0000 L CNN
-F 2 "Package_TO_SOT_THT:TO-92_Inline" H 5150 5925 50  0001 L CIN
+F 2 "Package_TO_SOT_THT:TO-92_Wide" H 5150 5925 50  0001 L CIN
 F 3 "https://www.onsemi.com/pub/Collateral/2N3903-D.PDF" H 4950 6000 50  0001 L CNN
 	1    4950 6000
@@
 F 0 "C15" H 13150 6150 50  0000 L CNN
 F 1 "200µF_200V" H 13000 6050 50  0000 L CNN
-F 2 "Capacitor_THT:CP_Radial_D18.0mm_P7.50mm" H 13638 5950 50  0001 C CNN
+F 2 "Capacitor_THT:CP_Radial_D22.0mm_P10.00mm_SnapIn" H 13638 5950 50  0001 C CNN
 F 3 "~" H 13600 6100 50  0001 C CNN
 	1    13600 6100
@@
 F 0 "C12" H 13150 5800 50  0000 L CNN
 F 1 "200µF_200V" H 13000 5700 50  0000 L CNN
-F 2 "Capacitor_THT:CP_Radial_D18.0mm_P7.50mm" H 13638 5600 50  0001 C CNN
+F 2 "Capacitor_THT:CP_Radial_D22.0mm_P10.00mm_SnapIn" H 13638 5600 50  0001 C CNN
 F 3 "~" H 13600 5750 50  0001 C CNN
 	1    13600 5750
@@
 F 0 "C11" V 13150 5250 50  0000 L CNN
 F 1 "100µF_200V" V 13250 5050 50  0000 L CNN
-F 2 "Capacitor_THT:CP_Radial_D18.0mm_P7.50mm" H 13038 5150 50  0001 C CNN
+F 2 "Capacitor_THT:CP_Radial_D16.0mm_P7.50mm" H 13038 5150 50  0001 C CNN
 F 3 "~" H 13000 5300 50  0001 C CNN
 	1    13000 5300
@@
 F 0 "C9" V 12250 4650 50  0000 L CNN
 F 1 "100µF_200V" V 12400 4500 50  0000 L CNN
-F 2 "Capacitor_THT:CP_Radial_D18.0mm_P7.50mm" H 12588 4550 50  0001 C CNN
+F 2 "Capacitor_THT:CP_Radial_D16.0mm_P7.50mm" H 12588 4550 50  0001 C CNN
 F 3 "~" H 12550 4700 50  0001 C CNN
 	1    12550 4700
@@
 $EndComp
 $Comp
-L pspice:DIODE D6
+L pspice:DIODE D5
 U 1 1 61C5A997
 P 13250 5100
-F 0 "D6" H 13250 5365 50  0000 C CNN
+F 0 "D5" H 13250 5365 50  0000 C CNN
 F 1 "FR154" H 13250 5274 50  0000 C CNN
 F 2 "Diode_THT:D_DO-41_SOD81_P10.16mm_Horizontal" H 13250 5100 50  0001 C CNN
@@
 F 0 "C7" V 11250 4650 50  0000 L CNN
 F 1 "100µF_200V" V 11400 4500 50  0000 L CNN
-F 2 "Capacitor_THT:CP_Radial_D18.0mm_P7.50mm" H 11588 4550 50  0001 C CNN
+F 2 "Capacitor_THT:CP_Radial_D16.0mm_P7.50mm" H 11588 4550 50  0001 C CNN
 F 3 "~" H 11550 4700 50  0001 C CNN
 	1    11550 4700
@@
 Wire Notes Line
 	8750 1500 8750 3700
+$Comp
+L Connector:Screw_Terminal_01x02 J1
+U 1 1 614916C3
+P 5500 2150
+F 0 "J1" H 5500 1950 50  0001 C CNN
+F 1 "Vin_cnt" H 5500 1900 50  0000 C CNN
+F 2 "TerminalBlock:TerminalBlock_Altech_AK300-2_P5.00mm" H 5500 2150 50  0001 C CNN
+F 3 "~" H 5500 2150 50  0001 C CNN
+	1    5500 2150
+	-1   0    0    1
+$EndComp
+Wire Wire Line
+	5850 2050 5700 2050
+$Comp
+L power:GND1 #PWR023
+U 1 1 6149DF93
+P 5700 2150
+F 0 "#PWR023" H 5700 1900 50  0001 C CNN
+F 1 "GND1" H 5705 1977 50  0000 C CNN
+F 2 "" H 5700 2150 50  0001 C CNN
+F 3 "" H 5700 2150 50  0001 C CNN
+	1    5700 2150
+	1    0    0    -1
+$EndComp
 $EndSCHEMATC

Commit message: up pcbs
Signed-off-by: fgl27 <fglfgl27@gmail.com>
Parts:
- added L2: 100µ, Inductor_THT:L_Axial_L5.0mm_D3.6mm_P10.00mm_Horizontal_Murata_BL01RN1A2A2, symbol pspice:INDUCTOR
- added R12: 80kΩ, Resistor_THT:R_Axial_DIN0207_L6.3mm_D2.5mm_P10.16mm_Horizontal, symbol Device:R
- R7: value 50kΩ -> 100kΩ
Connections:
- net at C12.1, J2.1 (Pin_1), R20.1: now also L2.2; no longer C11.1, D5.2 (A)
- net GND1 renamed GND
- net GND: now also R12.2; no longer J1.1 (Pin_1), POT1.3
- net GND2 renamed GNDA
- net GNDA: no longer C6.2, Q7.3 (C)
- new net: POT1.3, R12.1
- new net: C11.1, D5.2 (A), L2.1
- new net: C6.2, Q7.3 (C)
- new net GNDREF: J1.1 (Pin_1)
Other:
- moved on the sheet: C12, C15, R18, R20, R21, R22, TRIM_POT2

Commit message: up pcbs
Signed-off-by: fgl27 <fglfgl27@gmail.com>
Other:
- note added: "GND pertence a fonte de 12V\n\nGNDA pertence a fonte de 24V\n\nGND e GNDA não tem conexão física\n\nO GNDA do Estagio 4. Boost, preferencialmente deve estar a uma distância do\nGNDA do estagio 3, para evitar ruídos gerados pela corrente alta do boost"
- note removed: "GND1 pertence a fonte de 12V\n\nGND2 pertence a fonte de 24V\n\nGND1 e GND2 não tem conexão física\n\nO GND2 do Estagio 4. Boost, preferencialmente deve estar a uma distância do\nGND2 do estagio 3, para evitar ruídos gerados pela corrente alta do boost"
Changed lines of the file:
@@
 	9500 5750 9900 5750
 Text Notes 2250 9200 0    98   ~ 0
-GND1 pertence a fonte de 12V\n\nGND2 pertence a fonte de 24V\n\nGND1 e GND2 não tem conexão física\n\nO GND2 do Estagio 4. Boost, preferencialmente deve estar a uma distância do\nGND2 do estagio 3, para evitar ruídos gerados pela corrente alta do boost
+GND pertence a fonte de 12V\n\nGNDA pertence a fonte de 24V\n\nGND e GNDA não tem conexão física\n\nO GNDA do Estagio 4. Boost, preferencialmente deve estar a uma distância do\nGNDA do estagio 3, para evitar ruídos gerados pela corrente alta do boost
 Text Notes 2800 7550 0    59   ~ 0
 O estagio de amplificação\nFaz com que o sinal da saída do opto\nfique com valor de tensão de 12V\ne mais definido/quadrado possível

Commit message: up pcb
Signed-off-by: fgl27 <fglfgl27@gmail.com>
Parts:
- L2: value 100µ -> 1mH
Changed lines of the file:
@@
 P 13900 5300
 F 0 "L2" H 13900 5515 50  0000 C CNN
-F 1 "100µ" H 13900 5424 50  0000 C CNN
+F 1 "1mH" H 13900 5424 50  0000 C CNN
 F 2 "Inductor_THT:L_Axial_L5.0mm_D3.6mm_P10.00mm_Horizontal_Murata_BL01RN1A2A2" H 13900 5300 50  0001 C CNN
 F 3 "~" H 13900 5300 50  0001 C CNN
