File: boost_311v/boost_311v.kicad_pcb (KiCad board)
At the start: 2 copper layers, 59 parts, among them J1 Vin_cnt, J2 VO, J3 Vin_boost, Q1 BC556, Q2 PN2222A, Q3 PN2222A, Q4 PN2222A, Q5 IRFP260, Q6 2N3904, Q7 2N3906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

Commit message: up pcbs
Signed-off-by: fgl27 <fglfgl27@gmail.com>
Parts:
- added L2: 100µ, Inductor_THT:L_Axial_L5.0mm_D3.6mm_P10.00mm_Horizontal_Murata_BL01RN1A2A2, F.Cu at (86.4, 145.7)
- added R12: 80kΩ, Resistor_THT:R_Axial_DIN0207_L6.3mm_D2.5mm_P10.16mm_Horizontal, F.Cu at (143.0, 117.0)
- R7: value 50kΩ -> 100kΩ
- moved R5 2.49 mm to (141.4, 120.7)
Connections:
- net GND2 renamed GNDA
- C10 pad 1: GND1 -> GND
- C12 pad 1: Net-(C11-Pad1) -> Net-(C12-Pad1)
- C4 pad 2: GND1 -> GND
- C5 pad 2: GND1 -> GND
- C8 pad 2: GND1 -> GND
- J1 pad 1: GND1 -> GND
- J2 pad 1: Net-(C11-Pad1) -> Net-(C12-Pad1)
- POT1 pad 3: GND1 -> Net-(POT1-Pad3)
- Q2 pad 1: GND1 -> GND
- R16 pad 2: GND1 -> GND
- R20 pad 1: Net-(C11-Pad1) -> Net-(C12-Pad1)
- R5 pad 1: GND1 -> GND
- U4 pad 4: GND1 -> GND
- U5 pad 1: GND1 -> GND
Routing:
- net GND1: track 160.2 -> 0.00 mm
- net GND: track 0.00 -> 145.8 mm
- net Net-(C12-Pad1): track 0.00 -> 70.6 mm
- net Net-(C11-Pad1): track 61.8 -> 16.5 mm
- net Net-(POT1-Pad3): track 0.00 -> 26.8 mm
- net Net-(R5-Pad2): track 7.15 -> 10.8 mm
