File: pwm_protecao/pwm_protecao.sch (KiCad schematic (older format))
At the start: 28 parts, among them Q1 BC556, Q2 PN2222A, Q3 2N3904, Q4 2N3906, Q5 IRLZ44N, Q6 2N3904, Q7 2N3906, U1 4N25, U4 LF357, U5 NE555

Commit message: Up pcb
Signed-off-by: fgl27 <fglfgl27@gmail.com>
Parts:
- removed POT1: 200kΩ, Potentiometer_THT:Potentiometer_Alps_RK163_Single_Horizontal, symbol Device:R_POT
- removed Q1: BC556, Package_TO_SOT_THT:TO-92_Wide, symbol Transistor_BJT:BC556
- removed Q2: PN2222A, Package_TO_SOT_THT:TO-92_Inline, symbol Transistor_BJT:PN2222A
- removed R1, R2: 1kΩ, Resistor_THT:R_Axial_DIN0207_L6.3mm_D2.5mm_P10.16mm_Horizontal, symbol Device:R
- removed R15, R9: 10kΩ, Resistor_THT:R_Axial_DIN0207_L6.3mm_D2.5mm_P10.16mm_Horizontal, symbol Device:R
- removed R16: 100kΩ, Resistor_THT:R_Axial_DIN0207_L6.3mm_D2.5mm_P10.16mm_Horizontal, symbol Device:R
- removed R8: 470Ω, Resistor_THT:R_Axial_DIN0207_L6.3mm_D2.5mm_P10.16mm_Horizontal, symbol Device:R
- removed U4: LF357, Package_DIP:DIP-8_W7.62mm_LongPads, symbol Amplifier_Operational:LF357
- added D3, D4: 1N4007, Diode_THT:D_DO-41_SOD81_P10.16mm_Horizontal, symbol Diode:1N4007
- added RV1: 100kΩ, Potentiometer_THT:Potentiometer_Alps_RK163_Single_Horizontal, symbol Device:R_POT
- C4: value 10nF -> 100nF
- C5: value 333pF -> 571pF
- R3: value 100Ω -> 330Ω
- R5: value 220Ω -> 470Ω
Connections:
- net PWM: now also U5.3 (Q)
- net at U5.7 (DIS): now also R14.2, D3.1 (K), D4.2 (A)
- net F_Serra: no longer names the net of C5.1, U5.2 (TR), U5.6 (THR)
- net F_Serra: now also RV1.2
- new net: D4.1 (K), RV1.1
- new net: D3.2 (A), RV1.3
Other:
- note added: "1. PWMm - F ≈ 19kHz - Duty 10 a 100%"
- note added: "3.1 Proteções e acionamento MOSFET"
- note added: "3.2 Proteções e acionamento MOSFET"
- note added: "Ajustando o controle / potenciômetro se ajusta o Duty."
- note added: "Caso a frequência necessária, impeça o uso do optocoupler, use o isolamento com diodo\nuse diodos com tensão reversa de pelo menos 100V"
- note removed: "1. Geração dente de serra, 19kHz"
- note removed: "2. Comparador - Amplificação - PWM - duty 0 até 83%"
- note removed: "3.1 Isolamento e acionamento MOSFET"
- note removed: "3.2 Isolamento e acionamento MOSFET"
- note removed: "Como o circuito foi desenvolvido para demostrar funcionamento de um boost\no Duty foi limitado a no máximo 83%, impedindo assim colocar a fonte em curto\n\nCaso a frequência necessária, impeça o uso do optocoupler, use o isolamento com diodo\nuse diodos com tensão reversa de pelo menos 100V"
- note removed: "O Duty é limitado em no máximo ≈ 83%\nImpedindo assim colocar a fonte em curto\nAjustável usando o Controle / potenciômetro"
- moved on the sheet: C4, C5, C8, D1, D2, Q3, Q4, Q5, Q6, Q7, R14, R3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

Commit message: Up pcbs
Signed-off-by: fgl27 <fglfgl27@gmail.com>
Other:
- note added: "Felipe Leon - 2021"
Changed lines of the file:
@@
 Text Notes 3850 3000 0    79   ~ 0
 Ajustando o controle / potenciômetro se ajusta o Duty.
+Text Notes 7300 6350 0    79   ~ 0
+Felipe Leon - 2021
 $EndSCHEMATC

Commit message: Up pcb
Signed-off-by: fgl27 <fglfgl27@gmail.com>
Parts:
- removed Q6: 2N3904, Package_TO_SOT_THT:TO-92_Inline, symbol Transistor_BJT:2N3904
- removed Q7: 2N3906, Package_TO_SOT_THT:TO-92_Inline, symbol Transistor_BJT:2N3906
- removed R5, R6: 470Ω, Resistor_THT:R_Axial_DIN0207_L6.3mm_D2.5mm_P10.16mm_Horizontal, symbol Device:R
- removed U1: 4N25, Package_DIP:DIP-6_W7.62mm, symbol Isolator:4N25
- added C1, C3: 100nF, Capacitor_THT:C_Disc_D7.5mm_W5.0mm_P5.00mm, symbol pspice:CAP
- added L1: 1,5µH, symbol pspice:INDUCTOR
- added R1: 1kΩ, Resistor_THT:R_Axial_DIN0207_L6.3mm_D2.5mm_P10.16mm_Horizontal, symbol Device:R
Connections:
- net +12V: now also D1.2 (A), C3.1, L1.1; no longer Q3.3 (C), Q5.2 (D)
- net GND: now also Q5.3 (S), C1.2, C3.2; no longer R3.1
- net MOS_Gate: now also Q5.1 (G), R7.2; no longer Q3.1 (E), Q4.1 (E), R7.1
- net at Q3.2 (B), Q4.2 (B), R4.1: now also R1.2; no longer D2.1 (K)
- new net: D2.1 (K), R1.1
- new net: Q3.1 (E), Q4.1 (E), R7.1
- new net: C1.1, L1.2, Q3.3 (C)
- new net: Q5.2 (D), R3.1
Other:
- note added: "1. PWMm - F ≈ 19kHz - Duty 18 a 100%"
- note added: "2 Proteções e acionamento MOSFET\nBaseado no Bipolar Totem-Pole Driver"
- note added: "3. MOSFET - para demonstrar funcionamento"
- note removed: "1. PWMm - F ≈ 19kHz - Duty 10 a 100%"
- note removed: "3.1 Proteções e acionamento MOSFET"
- note removed: "3.2 Proteções e acionamento MOSFET"
- note removed: "4. MOSFET - para demonstrar funcionamento"
- note removed: "Caso a frequência necessária, impeça o uso do optocoupler, use o isolamento com diodo\nuse diodos com tensão reversa de pelo menos 100V"
- moved on the sheet: D1, D2, Q3, Q4, Q5, R3, R4, R7

Commit message: UP ocbs
Signed-off-by: fgl27 <fglfgl27@gmail.com>
Parts:
- removed C3: 100nF, Capacitor_THT:C_Disc_D7.5mm_W5.0mm_P5.00mm, symbol pspice:CAP
- removed D2: 1N4007, Diode_THT:D_DO-41_SOD81_P10.16mm_Horizontal, symbol Diode:1N4007
- removed L1: 1,5µH, symbol pspice:INDUCTOR
Connections:
- net +12V: now also C1.1, Q3.3 (C)
- net PWM: now also R1.1
Changed lines of the file:
@@
 	8100 3450 8100 5900
-Wire Wire Line
-	2000 5200 2000 5100
-Wire Wire Line
-	2000 4200 2000 4600
-Connection ~ 2000 4200
-Wire Wire Line
-	2000 4200 3200 4200
 Wire Wire Line
 	2900 4750 2750 4750
 Wire Wire Line
 	3350 5200 3850 5200
-Connection ~ 3350 5200
 Wire Wire Line
 	3350 5150 3350 5200
@@
 	3850 4350 3850 4200
 Wire Wire Line
-	3700 4200 3850 4200
-$Comp
-L pspice:INDUCTOR L1
-U 1 1 61455D72
-P 3450 4200
-F 0 "L1" H 3450 4415 50  0000 C CNN
-F 1 "1,5µH" H 3450 4324 50  0000 C CNN
-F 2 "" H 3450 4200 50  0001 C CNN
-F 3 "~" H 3450 4200 50  0001 C CNN
-	1    3450 4200
-	1    0    0    -1
-$EndComp
-Wire Wire Line
 	3850 5200 3850 5150
 Connection ~ 3850 5200
@@
 	1    0    0    -1
 $EndComp
-$Comp
-L pspice:CAP C3
-U 1 1 61450024
-P 2000 4850
-F 0 "C3" H 2100 5000 50  0000 L CNN
-F 1 "100nF" H 2100 4750 50  0000 L CNN
-F 2 "Capacitor_THT:C_Disc_D7.5mm_W5.0mm_P5.00mm" H 2000 4850 50  0001 C CNN
-F 3 "~" H 2000 4850 50  0001 C CNN
-	1    2000 4850
-	1    0    0    -1
-$EndComp
 Wire Wire Line
 	5100 4200 5100 4500
@@
 Text Label 4400 4750 0    59   ~ 0
 MOS_Gate
-Text Label 2450 4750 2    59   ~ 0
+Text Label 2750 4750 2    59   ~ 0
 PWM
-$Comp
-L Diode:1N4007 D2
-U 1 1 6138DCD7
-P 2600 4750
-F 0 "D2" H 2600 4533 50  0000 C CNN
-F 1 "1N4007" H 2600 4624 50  0000 C CNN
-F 2 "Diode_THT:D_DO-41_SOD81_P10.16mm_Horizontal" H 2600 4575 50  0001 C CNN
-F 3 "http://www.vishay.com/docs/88503/1n4001.pdf" H 2600 4750 50  0001 C CNN
-	1    2600 4750
-	-1   0    0    1
-$EndComp
 $Comp
 L Device:R R4
@@
 L power:+12V #PWR013
 U 1 1 615273D8
-P 2000 4200
-F 0 "#PWR013" H 2000 4050 50  0001 C CNN
-F 1 "+12V" H 2015 4373 50  0000 C CNN
-F 2 "" H 2000 4200 50  0001 C CNN
-F 3 "" H 2000 4200 50  0001 C CNN
-	1    2000 4200
+P 5100 4200
+F 0 "#PWR013" H 5100 4050 50  0001 C CNN
+F 1 "+12V" H 5115 4373 50  0000 C CNN
+F 2 "" H 5100 4200 50  0001 C CNN
+F 3 "" H 5100 4200 50  0001 C CNN
+	1    5100 4200
 	1    0    0    -1
 $EndComp
@@
 Wire Wire Line
 	3850 4200 5100 4200
-Connection ~ 3850 4200
 Wire Notes Line
 	1700 3450 1700 5900
@@
 Wire Notes Line
 	1700 3450 5500 3450
-Wire Wire Line
-	2000 5200 3350 5200
+Connection ~ 5100 4200
 $EndSCHEMATC
