File: pwm_new/boost_311v.kicad_pcb (KiCad board)
At the start: 2 copper layers, 27 parts, among them J1 Vin_cnt, J2 Carga, J3 Vin_boost, Q1 BC548, Q2 BC556, Q3 PN2222A, Q4 PN2222A, Q5 IRFP260, U3 4N25, U5 NE555

Commit message: Up pcb
Signed-off-by: fgl27 <fglfgl27@gmail.com>
Parts:
- moved POT1 44.5 mm to (128.0, 126.5), turned to 0 degrees
- moved C4 34.0 mm to (94.0, 128.0), turned to 90 degrees
- moved D1 33.2 mm to (117.9, 128.5), turned to 90 degrees
- moved J1 30.9 mm to (89.4, 104.6), turned to 180 degrees
- moved D2 19.9 mm to (117.9, 114.8)
- moved R8 19.5 mm to (113.3, 107.7), turned to 270 degrees
- moved U3 14.9 mm to (88.4, 128.0)
- moved HS1 14.4 mm to (78.7, 188.5)
- moved R17 11.9 mm to (101.6, 144.3)
- moved J2 11.9 mm to (63.0, 166.1)
- moved C16 11.9 mm to (111.8, 154.9)
- moved C5 11.9 mm to (94.0, 119.4)
- moved C6 11.9 mm to (76.2, 151.4)
- moved C8 11.9 mm to (106.7, 111.3)
- moved J3 11.9 mm to (116.3, 167.6)
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Connections:
- D1 pad 2: Net-(C5-Pad1) -> Net-(D1-Pad2)
- D2 pad 1: Net-(C5-Pad1) -> Net-(D1-Pad2)
- R8 pad 2: Net-(C5-Pad1) -> Net-(D1-Pad2)
- U5 pad 7: Net-(C5-Pad1) -> Net-(D1-Pad2)
Routing:
- net Net-(C5-Pad1): track 78.4 -> 36.7 mm
- net +12V: track 82.8 -> 56.9 mm
- net Net-(D1-Pad2): track 0.00 -> 16.2 mm
- net Net-(D2-Pad2): track 9.01 -> 22.0 mm
- net Net-(C4-Pad1): track 29.9 -> 17.1 mm
- net Net-(R5-Pad2): track 14.7 -> 3.05 mm
- net +12VA: track 135.8 -> 143.3 mm
- net GND1: track 50.7 -> 46.3 mm
- net Net-(D1-Pad1): track 9.65 -> 12.2 mm
- net /PWM: track 16.0 -> 17.8 mm
- net Net-(R11-Pad1): track 6.10 -> 6.81 mm
- net Net-(Q3-Pad2): track 3.98 -> 4.57 mm
Other:
- board text added: "Carga 12V"
- board text added: "Controle 12V"
- board text added: "Mosfet 12V"
