File: pwm_new/boost_311v.sch (KiCad schematic (older format))
At the start: 27 parts, among them J1 Vin_cnt, J2 Carga, J3 Vin_boost, Q1 BC548, Q2 BC556, Q3 PN2222A, Q4 PN2222A, Q5 IRFP260, U3 4N25, U5 NE555

Commit message: Up pcb
Signed-off-by: fgl27 <fglfgl27@gmail.com>
Connections:
- net at C5.1, POT1.2, U5.2 (TR)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: no longer D1.2 (A), D2.1 (K), R8.2, U5.7 (DIS)
- new net: D1.2 (A), D2.1 (K), R8.2, U5.7 (DIS)
Other:
- note added: "1.PWM - F ≈ 19 kHz - Duty ≈ 18 até 100%"
- note added: "3. Mosfet e carga"
- note removed: "1. Onda dente de serra, F ≈ 19 kHz - Duty 18 até 100%"
- note removed: "2. Mosfet e carga"
- note removed: "3. Isolação PWM, acionamento e proteção MOSFET"
- moved on the sheet: C16, C4, C5, C6, C8, D1, D2, HS1, POT1, Q1, Q2, Q3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
